Commit message: initial commit

File: description/lidar.xacro (robot description, xacro)
@@ -4,10 +4,10 @@
         <parent link="chassis"/>
         <child link="laser_frame"/>
-        <origin xyz="0.3 0 0.12" rpy="0 0 0"/>
+        <origin xyz="0.224 0 0.12" rpy="0 0 ${pi/2}"/>
     </joint>
     <link name="laser_frame">
         <visual>
             <geometry>
-                <cylinder radius="0.05" length="0.04"/>
+                <cylinder radius="0.035" length="0.028"/>
             </geometry>
             <material name="red"/>
@@ -15,8 +15,8 @@
         <collision>
             <geometry>
-                <cylinder radius="0.05" length="0.04"/>
+                <cylinder radius="0.035" length="0.028"/>
             </geometry>
         </collision>
-        <xacro:inertial_cylinder mass="0.1" length="0.04" radius="0.05">
+        <xacro:inertial_cylinder mass="0.1" length="0.028" radius="0.03">
             <origin xyz="0 0 0" rpy="0 0 0"/>
         </xacro:inertial_cylinder>

File: description/robot_core.xacro (robot description, xacro)
@@ -32,9 +32,9 @@
         <parent link="base_link"/>
         <child link="chassis"/>
-        <origin xyz="-0.1 0 0"/>
+        <origin xyz="-0.06 0 0"/>
     </joint>
     <link name="chassis">
         <visual>
-            <origin xyz="0.15 0 0.05"/>
+            <origin xyz="0.12 0 0.06"/>
             <geometry>
                 <cylinder radius="0.2" length="0.1"/>
@@ -43,11 +43,11 @@
         </visual>
         <collision>
-            <origin xyz="0.15 0 0.05"/>
+            <origin xyz="0.12 0 0.06"/>
             <geometry>
-                <cylinder radius="0.2" length="0.1"/>
+                <cylinder radius="0.225" length="0.1"/>
             </geometry>
         </collision>
-        <xacro:inertial_cylinder mass="5.0" radius="0.2" length="0.1">
-            <origin xyz="0.15 0 0.05" rpy="0 0 0"/>
+        <xacro:inertial_cylinder mass="5.0" radius="0.225" length="0.1">
+            <origin xyz="0.12 0 0.06" rpy="0 0 0"/>
         </xacro:inertial_cylinder>
     </link>
@@ -59,5 +59,5 @@
         <parent link="base_link"/>
         <child link="left_wheel"/>
-        <origin xyz="0 0.15 0" rpy="-${pi/2} 0 0" />
+        <origin xyz="0 0.146 0" rpy="-${pi/2} 0 0" />
         <!-- XYZ la vi tri banh xe cach tam base link, xoay cylinder banh1 goc -pi/2(90do)-->
         <axis xyz="0 0 1"/>
@@ -67,5 +67,5 @@
         <visual>
             <geometry>
-                <cylinder radius="0.05" length="0.04"/>
+                <cylinder radius="0.0325" length="0.026"/>
             </geometry>
             <material name="blue"/>
@@ -73,8 +73,8 @@
         <collision>
             <geometry>
-                <cylinder radius="0.05" length="0.04"/>
+                <cylinder radius="0.0325" length="0.026"/>
             </geometry>
         </collision>
-        <xacro:inertial_cylinder mass="0.1" length="0.04" radius="0.05">
+        <xacro:inertial_cylinder mass="0.1" length="0.026" radius="0.0325">
             <origin xyz="0 0 0" rpy="0 0 0"/>
         </xacro:inertial_cylinder>
@@ -87,5 +87,5 @@
         <parent link="base_link"/>
         <child link="right_wheel"/>
-        <origin xyz="0 -0.15 0" rpy="${pi/2} 0 0" />
+        <origin xyz="0 -0.146 0" rpy="${pi/2} 0 0" />
         <axis xyz="0 0 -1"/>
     </joint>
@@ -93,5 +93,5 @@
         <visual>
             <geometry>
-                <cylinder radius="0.05" length="0.04"/>
+                <cylinder radius="0.0325" length="0.026"/>
             </geometry>
             <material name="blue"/>
@@ -99,8 +99,8 @@
         <collision>
             <geometry>
-                <cylinder radius="0.05" length="0.04"/>
+                <cylinder radius="0.0325" length="0.026"/>
             </geometry>
         </collision>
-        <xacro:inertial_cylinder mass="0.1" length="0.04" radius="0.05">
+        <xacro:inertial_cylinder mass="0.1" length="0.026" radius="0.0325">
             <origin xyz="0 0 0" rpy="0 0 0"/>
         </xacro:inertial_cylinder>
@@ -113,10 +113,10 @@
         <parent link="chassis"/>
         <child link="caster_wheel"/>
-        <origin xyz="0.3 0 0"/>
+        <origin xyz="0.24 0 0"/>
     </joint>
     <link name="caster_wheel">
         <visual>
             <geometry>
-                <sphere radius="0.05"/>
+                <sphere radius="0.0325"/>
             </geometry>
             <material name="black"/>
@@ -124,8 +124,8 @@
         <collision>
             <geometry>
-                <sphere radius="0.05"/>
+                <sphere radius="0.0325"/>
             </geometry>
         </collision>
-        <xacro:inertial_sphere mass="0.2" radius="0.05">
+        <xacro:inertial_sphere mass="0.2" radius="0.0325">
             <origin xyz="0 0 0" rpy="0 0 0"/>
         </xacro:inertial_sphere>
